Commit message: feat: solve unseen mazes with lidar sensing and closed-loop odometry
The brain previously read every wall from disk, flooded once and fired the
whole path in a burst. The robot executed a known solution; it discovered
nothing. This adds an explorer that starts knowing only the grid size, the
start cell and the goal, and learns the rest from a laser scanner.

The maze definition splits in two. maze_spec.json carries geometry, start and
goal but no walls; maze_truth.json carries the walls and is read only by the
simulated sensor, the viz and the baseline brain. spec.read_public raises on a
file containing walls, so wiring a blind component to the truth file fails
loudly instead of quietly handing it the answer.

BeliefMaze gives every wall three states. Read optimistically (unknown = open)
the flood-fill gradient pulls the robot into unexplored ground; read
pessimistically (unknown = wall) it only commits to verified passages. Optimism
is a property of the object, so flood_fill and planner consume a belief
unchanged. Explorer drives three phases: search to the goal, return home still
sensing, then a speed run on the learned map.

Exploration inverts the old architecture. The brain cannot know move n+1 until
the robot has arrived at cell n and read there, so it runs in strict lockstep.
Waiting for the next scan is not enough: the lidar publishes on its own clock,
so a scan can arrive after arrival but be computed from the previous pose, and
the brain then files the wrong cell's walls. settled_reading waits for
consecutive scans to agree instead, which needs no cooperation from the sensor.

Motion closes the loop. motion:=velocity publishes /cmd_vel and reads /odom;
motion:=pose keeps the teleport for recording. Three things had to be right:
odom is anchored at the robot's spawn, not the world origin, so it needs an
explicit transform (without it the belief walls off the start cell); turn
targets must be absolute or every turn keeps its own error; and holding a
heading by turning mid-drive curves the path, so lateral offset is corrected
against the side walls.

Real Gazebo gpu_lidar is available behind lidar:=gz. It needs the Ogre render
engine, which does not load on a GPU-less host, so raycast_lidar is the default
and the sensors system is opt-in via generate_maze --sensors.

gazebo_sync_brain is untouched and kept as the omniscient baseline.

Tests cover the policy offline against an oracle sensor over 30 seeds, plus a
hand-built lure maze, because generated mazes never trigger backtracking and
that path would otherwise be untested.

File: src/micromouse/description/micromouse.urdf.xacro (robot description, xacro)
@@ -4,4 +4,8 @@
        wheel_radius=0.04, wheel_separation=0.13. Spawn at z=0.04 so the
        wheels rest on the ground. -->
+  <!-- The real Gazebo LiDAR is off by default. gpu_lidar needs the Ogre render
+       engine, which does not load on a GPU-less host, so the default sensor is
+       the raycast_lidar node. Turn this on with lidar:=gz. -->
+  <xacro:arg name="use_lidar" default="false"/>
   <link name="base_link">
     <visual>
@@ -84,4 +88,53 @@
     <origin xyz="0.045 0 -0.02" rpy="0 0 0"/>
   </joint>
+  <!-- lidar mount (always present so TF is stable; the sensor itself is
+       conditional) -->
+  <link name="lidar_link">
+    <visual>
+      <geometry><cylinder length="0.01" radius="0.015"/></geometry>
+      <material name="lidar"><color rgba="0.8 0.2 0.2 1"/></material>
+    </visual>
+    <inertial>
+      <mass value="0.01"/>
+      <inertia ixx="0.0000006" ixy="0" ixz="0"
+               iyy="0.0000006" iyz="0" izz="0.0000011"/>
+    </inertial>
+  </link>
+  <joint name="lidar_joint" type="fixed">
+    <parent link="base_link"/>
+    <child link="lidar_link"/>
+    <origin xyz="0 0 0.025" rpy="0 0 0"/>
+  </joint>
+  <xacro:if value="$(arg use_lidar)">
+    <gazebo reference="lidar_link">
+      <sensor name="lidar" type="gpu_lidar">
+        <topic>/scan</topic>
+        <gz_frame_id>lidar_link</gz_frame_id>
+        <update_rate>20</update_rate>
+        <always_on>true</always_on>
+        <visualize>false</visualize>
+        <lidar>
+          <scan>
+            <horizontal>
+              <samples>72</samples>
+              <resolution>1</resolution>
+              <min_angle>-3.141593</min_angle>
+              <max_angle>3.141593</max_angle>
+            </horizontal>
+          </scan>
+          <range>
+            <min>0.02</min>
+            <max>4.0</max>
+            <resolution>0.01</resolution>
+          </range>
+          <noise>
+            <type>gaussian</type>
+            <mean>0.0</mean>
+            <stddev>0.0</stddev>
+          </noise>
+        </lidar>
+      </sensor>
+    </gazebo>
+  </xacro:if>
   <!-- gz friction: grippy wheels, slippery caster -->
   <gazebo reference="left_wheel">
